Commit message: Update encoder and fix

File: intelijet_v2_ws/src/pps/urdf/scanner_housing.urdf (robot description, URDF)
Before this commit: robot scanner, 4 links, 3 joints
Links:
- link LMS-511: geometry visual box size=0.1 0.2 0.01
Joints:
- joint scan_to_scanner: origin xyz=0.08 0 0 rpy=0 0 0 -> xyz=0 0 0 rpy=0 0 1.57
- joint scanner_deploy_retract: axis 0 -1 0 -> -1 0  0; origin xyz=0 0 0.5 rpy=0 0 0 -> xyz=0 0 0 rpy=1.74 0 0

Commit message: update ui

File: intelijet_v2_ws/src/pps/urdf/scanner_housing.urdf (robot description, URDF)
Before this commit: robot scanner, 4 links, 3 joints
Links:
- link LMS-511: geometry visual box size=0.5 0.2 0.01
- link scanner_mount: geometry visual box size=0.05 0.4 0.05
Joints:
- joint scanner_deploy_retract: origin xyz=0 0 0 rpy=1.74 0 0 -> xyz=0 0 0 rpy=0 0 0

Commit message: update

File: intelijet_v2_ws/src/pps/urdf/scanner_housing.urdf (robot description, URDF)
Before this commit: robot scanner, 4 links, 3 joints
Joints:
- joint scan_to_scanner: origin xyz=0 0 0 rpy=0 0 1.57 -> xyz=0 0 0 rpy=0 0 0
- joint scanner_deploy_retract: axis -1 0  0 -> 0 1 0; origin xyz=0 0 0 rpy=0 0 0 -> xyz=0 0 0 rpy=0 -2.04 0

Commit message: update

File: intelijet_v2_ws/src/pps/urdf/scanner_housing.urdf (robot description, URDF)
Before this commit: robot scanner, 4 links, 3 joints
Joints:
- joint scanner_deploy_retract: origin xyz=0 0 0 rpy=0 -2.04 0 -> xyz=0 0 0.75 rpy=0 -2.04 0

Commit message: ajust home position of housing in scanner_housing.urdf

File: intelijet_v2_ws/src/pps/urdf/scanner_housing.urdf (robot description, URDF)
Before this commit: robot scanner, 4 links, 3 joints
Links:
- link LMS-511: geometry visual box size=0.05 0.05 0.05
- link scanner_mount: geometry visual box size=0.2 0.01 0.01
Joints:
- joint scanner_deploy_retract: origin xyz=0 0 0.75 rpy=0 -2.04 0 -> xyz=0 0 0.75 rpy=0 -1.780236 0
- joint scanner_to_mount: origin xyz=0 0 0 rpy=0 0 0 -> xyz=0.276 0 0 rpy=0 0 0
