Commit message: [pps] Fix stale prescan in auto-compare, unify with manual compare flow
Auto-compare (after Post-Scan) relied on ROS param
/runtime/last_prescan_path, which was only ever written once at UI
startup - any Pre-Scan taken later in the session was invisible to it,
so compare could silently run against a stale/wrong Pre-Scan file.

ScanPipelineWorker now tracks the live prescan path itself and passes
explicit prescan/postscan paths to App, which runs auto-compare through
the same CompareWorker/`/compare_cloud_manual` pipeline manual compare
already used - removing the stale ROS-param path entirely. Falls back
to scanning the job folder for the newest Pre-Scan file if the tracked
path is missing/not yet written. Auto-compare takes priority over an
in-flight manual compare (its result is discarded if pre-empted), and
both flows now serialize through a single in-flight guard, closing a
pre-existing race where isManualCompare/current_post_scan_path could
mis-tag which job a compared-cloud result belonged to.

Removes the now-dead /compare_cloud action server, CompareBaseClient,
and the HMI START_COMPARE command path.

Co-Authored-By: Claude Sonnet 5 <noreply@anthropic.com>

File: intelijet_v2_ws/src/pps/urdf/scanner_housing.urdf (robot description, URDF)
Before this commit: robot scanner, 4 links, 3 joints
Joints:
- joint scanner_deploy_retract: origin xyz=0 0 0.75 rpy=0 -1.780236 0 -> xyz=0 0 1.3 rpy=0 -1.780236 0
